Commit message: training with sphere working

File: assets/urdf/pentapede/urdf/pentapede.urdf (robot description, URDF)
Before this commit: robot pentapede, 86 links, 85 joints
Links:
- removed link wx250s/ee_arm_link
- link wx250s/gripper_link: geometry collision mesh filename=package://pentapede/meshes/wx250s_7_gripper.stl scale=0.001 0.001 0.001; visual box size=0.01 0.01 0.01
Joints:
- removed joint ee_arm
